Commit message: add base_footprint in urdf

File: SC-22_src_0723/ForROS_description/urdf/ForROS.xacro (robot description, xacro)
@@ -4,4 +4,5 @@
 <xacro:include filename="$(find ForROS_description)/urdf/ForROS.trans" />
 <xacro:include filename="$(find ForROS_description)/urdf/ForROS.gazebo" />
+<link name="base_footprint"/>
 <link name="base_link">
   <inertial>
@@ -11,5 +12,5 @@
   </inertial>
   <visual>
-    <origin xyz="0 0 0" rpy="0 0 0"/>
+    <origin xyz="0 0 -0.073005" rpy="0 0 0"/>
     <geometry>
       <mesh filename="file://$(find ForROS_description)/meshes/base_link.stl" scale="0.001 0.001 0.001"/>
@@ -145,20 +146,20 @@
 </link>
 <joint name="Rigid_Pi" type="fixed">
-  <origin xyz="-0.019 0.0045 0.098205" rpy="0 0 0"/>
+  <origin xyz="-0.019 0.0045 0.0252" rpy="0 0 0"/>
   <parent link="base_link"/>
   <child link="RaspberryPi_1"/>
 </joint>
 <joint name="Rigid_Camera" type="fixed">
-  <origin xyz="0.01243 0.043715 0.081725" rpy="0 0 0"/>
+  <origin xyz="0.01243 0.043715 0.00872" rpy="0 0 0"/>
   <parent link="base_link"/>
   <child link="Camera_link_1"/>
 </joint>
 <joint name="Rigid_Battery" type="fixed">
-  <origin xyz="0.0365 -0.037 0.075505" rpy="0 0 0"/>
+  <origin xyz="0.0365 -0.037 0.0025" rpy="0 0 0"/>
   <parent link="base_link"/>
   <child link="Battery_v1_1_1"/>
 </joint>
 <joint name="lidar_joint" type="continuous">
-  <origin xyz="0.0 0.03 0.083805" rpy="0 0 0"/>
+  <origin xyz="0.0 0.03 0.0108" rpy="0 0 0"/>
   <parent link="base_link"/>
   <child link="Lidar_link_1"/>
@@ -166,5 +167,5 @@
 </joint>
 <joint name="r_joint" type="continuous">
-  <origin xyz="0.0902 0.0 0.073005" rpy="0 0 0"/>
+  <origin xyz="0.0902 0.0 0.0" rpy="0 0 0"/>
   <parent link="base_link"/>
   <child link="Rwheel_link_1"/>
@@ -172,8 +173,13 @@
 </joint>
 <joint name="l_joint" type="continuous">
-  <origin xyz="-0.0902 0.0 0.073005" rpy="0 0 0"/>
+  <origin xyz="-0.0902 0.0 0.0" rpy="0 0 0"/>
   <parent link="base_link"/>
   <child link="Lwheel_link_1"/>
   <axis xyz="-1.0 0.0 0.0"/>
 </joint>
+<joint name="base_joint" type="fixed">
+  <origin xyz="0 0 0.073005"/>
+  <parent link="base_footprint"/>
+  <child link="base_link"/>
+</joint>
 </robot>

Commit message: Change link name

File: SC-22_src_0723/ForROS_description/urdf/ForROS.xacro (robot description, xacro)
@@ -25,5 +25,5 @@
   </collision>
 </link>
-<link name="RaspberryPi_1">
+<link name="RaspberryPi">
   <inertial>
     <origin xyz="0.000549946651029417 -0.023988893579614225 0.005680415420320897" rpy="0 0 0"/>
@@ -45,5 +45,5 @@
   </collision>
 </link>
-<link name="Camera_link_1">
+<link name="Camera_link">
   <inertial>
     <origin xyz="-0.01234464717368007 0.0007909573025063274 -0.010732269549067155" rpy="0 0 0"/>
@@ -65,5 +65,5 @@
   </collision>
 </link>
-<link name="Battery_v1_1_1">
+<link name="Battery">
   <inertial>
     <origin xyz="-0.036499999999999894 8.326672684688674e-17 0.0" rpy="0 0 0"/>
@@ -85,5 +85,5 @@
   </collision>
 </link>
-<link name="Lidar_link_1">
+<link name="Lidar_link">
   <inertial>
     <origin xyz="-0.005110778358159219 -0.00037745206548664076 0.014726243086830501" rpy="0 0 0"/>
@@ -105,5 +105,5 @@
   </collision>
 </link>
-<link name="Rwheel_link_1">
+<link name="Rwheel_link">
   <inertial>
     <origin xyz="0.009999999046325828 -4.0829913766993425e-16 -7.216449660063518e-16" rpy="0 0 0"/>
@@ -125,5 +125,5 @@
   </collision>
 </link>
-<link name="Lwheel_link_1">
+<link name="Lwheel_link">
   <inertial>
     <origin xyz="-0.00999999904632548 -2.4446522753376446e-16 -4.3021142204224816e-16" rpy="0 0 0"/>
@@ -148,20 +148,20 @@
   <origin xyz="-0.019 0.0045 0.0252" rpy="0 0 0"/>
   <parent link="base_link"/>
-  <child link="RaspberryPi_1"/>
+  <child link="RaspberryPi"/>
 </joint>
 <joint name="Rigid_Camera" type="fixed">
   <origin xyz="0.01243 0.043715 0.00872" rpy="0 0 0"/>
   <parent link="base_link"/>
-  <child link="Camera_link_1"/>
+  <child link="Camera_link"/>
 </joint>
 <joint name="Rigid_Battery" type="fixed">
   <origin xyz="0.0365 -0.037 0.0025" rpy="0 0 0"/>
   <parent link="base_link"/>
-  <child link="Battery_v1_1_1"/>
+  <child link="Battery"/>
 </joint>
 <joint name="lidar_joint" type="continuous">
   <origin xyz="0.0 0.03 0.0108" rpy="0 0 0"/>
   <parent link="base_link"/>
-  <child link="Lidar_link_1"/>
+  <child link="Lidar_link"/>
   <axis xyz="0.0 -0.0 -1.0"/>
 </joint>
@@ -169,5 +169,5 @@
   <origin xyz="0.0902 0.0 0.0" rpy="0 0 0"/>
   <parent link="base_link"/>
-  <child link="Rwheel_link_1"/>
+  <child link="Rwheel_link"/>
   <axis xyz="1.0 -0.0 -0.0"/>
 </joint>
@@ -175,5 +175,5 @@
   <origin xyz="-0.0902 0.0 0.0" rpy="0 0 0"/>
   <parent link="base_link"/>
-  <child link="Lwheel_link_1"/>
+  <child link="Lwheel_link"/>
   <axis xyz="-1.0 0.0 0.0"/>
 </joint>
